File: LumioV2.kicad_pcb (KiCad board)
At the start: 2 copper layers, 56 parts, among them J1 I2C POINT 1 - QWIIC, J10 MOTOR B, J11 Analog Input, J12 Analog Input, J13 Analog Input, J14 Analog Input, J15 Analog Input, J16 Analog Input, J17 Analog Input, J18 Analog Input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

Commit message: began routing
Parts:
- added C25: 100nF, Capacitor_SMD:C_0402_1005Metric_Pad0.74x0.62mm_HandSolder, F.Cu at (148.3, 64.5)
- added C26: 33pF, Capacitor_SMD:C_0402_1005Metric_Pad0.74x0.62mm_HandSolder, F.Cu at (122.4, 61.1)
- added C27: 33pF, Capacitor_SMD:C_0402_1005Metric_Pad0.74x0.62mm_HandSolder, F.Cu at (124.4, 61.1)
- added C28: 100nF, Capacitor_SMD:C_0402_1005Metric_Pad0.74x0.62mm_HandSolder, F.Cu at (256.0, 103.3)
- added C29: 100nF, Capacitor_SMD:C_0402_1005Metric_Pad0.74x0.62mm_HandSolder, F.Cu at (256.0, 105.3)
- added C30: 100nF, Capacitor_SMD:C_0402_1005Metric_Pad0.74x0.62mm_HandSolder, F.Cu at (259.2, 97.4)
- added C31: 100nF, Capacitor_SMD:C_0402_1005Metric_Pad0.74x0.62mm_HandSolder, F.Cu at (259.2, 99.4)
- added C32: 100nF, Capacitor_SMD:C_0402_1005Metric_Pad0.74x0.62mm_HandSolder, F.Cu at (259.2, 101.4)
- added C33: 100nF, Capacitor_SMD:C_0402_1005Metric_Pad0.74x0.62mm_HandSolder, F.Cu at (259.2, 103.3)
- added C34: 1uF, Capacitor_SMD:C_0402_1005Metric_Pad0.74x0.62mm_HandSolder, F.Cu at (138.4, 66.0)
- added C35: 1uF, Capacitor_SMD:C_0402_1005Metric_Pad0.74x0.62mm_HandSolder, F.Cu at (124.5, 63.1)
- added C36: 100nF, Capacitor_SMD:C_0402_1005Metric_Pad0.74x0.62mm_HandSolder, F.Cu at (140.4, 66.2)
- added C37: 100nF, Capacitor_SMD:C_0402_1005Metric_Pad0.74x0.62mm_HandSolder, F.Cu at (140.4, 65.0)
- added C98: 1uF, Capacitor_SMD:C_0402_1005Metric_Pad0.74x0.62mm_HandSolder, F.Cu at (137.2, 66.3)
- added C99: 1uF, Capacitor_SMD:C_0402_1005Metric_Pad0.74x0.62mm_HandSolder, B.Cu at (127.1, 60.6)
- added J19: Serial Pads, Connector_PinHeader_2.54mm:PinHeader_1x02_P2.54mm_Vertical, F.Cu at (123.7, 48.2)
- added J20: Conn_02x13_Odd_Even, Connector_PinHeader_2.54mm:PinHeader_2x13_P2.54mm_Horizontal, F.Cu at (154.0, 28.6)
- added J21: Conn_02x02_Odd_Even, Connector_PinHeader_2.54mm:PinHeader_2x02_P2.54mm_Vertical, F.Cu at (143.2, 69.3)
- added P1: USB_C_Plug_USB2.0, Connector_USB:USB_C_Receptacle_GCT_USB4105-xx-A_16P_TopMnt_Horizontal, B.Cu at (141.1, 30.9)
- added R2: 5.1K, Resistor_SMD:R_0805_2012Metric_Pad1.20x1.40mm_HandSolder, F.Cu at (254.7, 107.9)
- added R3: 27, Resistor_SMD:R_0805_2012Metric_Pad1.20x1.40mm_HandSolder, B.Cu at (140.9, 63.2)
- added R4: 27, Resistor_SMD:R_0805_2012Metric_Pad1.20x1.40mm_HandSolder, B.Cu at (140.9, 61.2)
- added SW1: SW_Push, Button_Switch_SMD:SW_SPST_PTS647_Sx50, F.Cu at (121.9, 67.5)
- added SW2: SW_Push, Button_Switch_SMD:SW_SPST_PTS647_Sx50, F.Cu at (145.9, 51.8)
- added U4: RP2040, Package_DFN_QFN:QFN-56-1EP_7x7mm_P0.4mm_EP3.2x3.2mm, F.Cu at (133.5, 61.0)
- added U5: W25Q64JVXGIQ TR, Package_DFN_QFN:DFN-8-1EP_6x5mm_P1.27mm_EP4x4mm, F.Cu at (146.6, 59.0)
- added Y1: Crystal, Crystal:Crystal_SMD_HC49-SD, F.Cu at (114.5, 59.4)
- C10, C11, C12, C13, C14, C15, C8, C9: moved to B.Cu
- L1: footprint Inductor_THT:L_Radial_D21.0mm_P19.00mm -> Inductor_THT:L_Radial_D10.0mm_P5.00mm_Fastron_07M
- moved J8 98.5 mm to (200.9, 84.2), turned to 90 degrees
- moved C16 88.6 mm to (218.2, 141.9)
- moved C17 88.6 mm to (218.2, 143.9)
- moved C18 88.6 mm to (221.4, 130.1)
- moved C19 88.6 mm to (221.4, 132.1)
- moved C22 88.6 mm to (221.4, 138.0)
- moved C23 88.6 mm to (221.4, 140.0)
- moved C24 88.6 mm to (221.4, 141.9)
- moved C21 75.8 mm to (88.3, 42.7), turned to 180 degrees
- moved J3 66.5 mm to (69.0, 45.7), turned to 90 degrees
- moved R1 64.4 mm to (76.1, 84.8)
- moved J4 62.3 mm to (69.0, 61.1), turned to 90 degrees
- moved J18 61.6 mm to (157.9, 103.6), turned to -90 degrees
- moved J17 58.6 mm to (157.9, 98.1), turned to -90 degrees
- moved J11 58.4 mm to (157.8, 65.6), turned to -90 degrees
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Routing:
- net Net-(J5-Pin_40): track 0.00 -> 52.8 mm, vias 0 -> 3
- net Net-(J5-Pin_35): track 0.00 -> 52.3 mm, vias 0 -> 1
- net +3V3: track 0.00 -> 25.1 mm, vias 0 -> 1
- net Net-(U4-XOUT): track 0.00 -> 22.1 mm
- net Net-(J19-Pin_1): track 0.00 -> 19.8 mm, vias 0 -> 1
- net Net-(U4-~{QSPI_SS}): track 0.00 -> 18.1 mm
- net Net-(J19-Pin_2): track 0.00 -> 18.0 mm, vias 0 -> 1
- net Net-(U4-QSPI_SD1): track 0.00 -> 14.2 mm
- net Net-(U4-QSPI_SD2): track 0.00 -> 13.1 mm
- net Net-(U4-QSPI_SD3): track 0.00 -> 12.9 mm
- net Net-(U4-XIN): track 0.00 -> 12.1 mm
- net Net-(U4-QSPI_SCLK): track 0.00 -> 11.4 mm
- net +1V1: track 0.00 -> 10.9 mm
- net Net-(U4-QSPI_SD0): track 0.00 -> 8.78 mm
- net Net-(U4-RUN): track 0.00 -> 6.76 mm
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