File: LumioV2.kicad_sch (KiCad schematic)
At the start: 64 parts, among them J1 I2C POINT 1 - QWIIC, J10 MOTOR B, J11 Analog Input, J12 Analog Input, J13 Analog Input, J14 Analog Input, J15 Analog Input, J16 Analog Input, J17 Analog Input, J18 Analog Input, J19 Serial Pads, J2 I2C POINT 2 - QWIIC, J3 I2C POINT 3 - JST-PH, J4 I2C POINT 4 - JST-PH, J5 Raspi 5, J6 US Dist - Front, J7 US Dist - Back, J8 Display Connector, J9 MOTOR A, U1 LM2577T-ADJ/NOPB, U2 L298N, U3 MCP3008, U4 RP2040, U5 W25Q64JVXGIQ TR, Y1 Crystal

Commit message: smol changes
Parts:
- added P1: USB_C_Plug_USB2.0, symbol Connector:USB_C_Plug_USB2.0
Connections:
- net GND: now also C25.1, C26.1, C27.2, C28.1, U4.57 (GND), U5.4 (GND), U5.9, P1.A1 (GND), P1.A12 (GND), P1.B1 (GND), P1.B12 (GND)
- net at U4.46 (USB_DM): now also P1.A7 (D-)
- net at U4.47 (USB_DP): now also P1.A6 (D+)
- new net: P1.A4 (VBUS), P1.A9 (VBUS), P1.B4 (VBUS), P1.B9 (VBUS)
Other:
- moved on the sheet: J19
Changed lines of the file:
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@@
 	)
 	(junction
+		(at 363.22 60.96)
+		(diameter 0)
+		(color 0 0 0 0)
+	)
+	(junction
 		(at 63.5 171.45)
 		(diameter 0)
@@
 	)
 	(junction
+		(at 261.62 45.72)
+		(diameter 0)
+		(color 0 0 0 0)
+	)
+	(junction
 		(at 255.27 46.99)
 		(diameter 0)
@@
 	)
 	(junction
+		(at 304.8 45.72)
+		(diameter 0)
+		(color 0 0 0 0)
+	)
+	(junction
 		(at 213.36 46.99)
 		(diameter 0)
@@
 	(wire
 		(pts
+			(xy 339.09 149.86) (xy 340.36 149.86)
+		)
+		(stroke
+			(width 0)
+			(type default)
+		)
+	)
+	(wire
+		(pts
 			(xy 50.8 151.13) (xy 66.04 151.13)
 		)
@@
 	(wire
 		(pts
-			(xy 340.36 147.32) (xy 337.82 147.32)
-		)
-		(stroke
-			(width 0)
-			(type default)
-		)
-	)
-	(wire
-		(pts
 			(xy 207.01 41.91) (xy 209.55 41.91)
 		)
@@
 	(wire
 		(pts
+			(xy 330.2 41.91) (xy 330.2 99.06)
+		)
+		(stroke
+			(width 0)
+			(type default)
+		)
+	)
+	(wire
+		(pts
 			(xy 227.33 46.99) (xy 236.22 46.99)
 		)
@@
 	(wire
 		(pts
+			(xy 304.8 26.67) (xy 304.8 45.72)
+		)
+		(stroke
+			(width 0)
+			(type default)
+		)
+	)
+	(wire
+		(pts
 			(xy 100.33 118.11) (xy 151.13 118.11)
 		)
@@
 	(wire
 		(pts
+			(xy 325.12 101.6) (xy 340.36 101.6)
+		)
+		(stroke
+			(width 0)
+			(type default)
+		)
+	)
+	(wire
+		(pts
 			(xy 215.9 119.38) (xy 215.9 161.29)
 		)
@@
 	(wire
 		(pts
-			(xy 215.9 161.29) (xy 223.52 161.29)
+			(xy 304.8 60.96) (xy 363.22 60.96)
 		)
 		(stroke
@@
 	(wire
 		(pts
-			(xy 340.36 161.29) (xy 353.06 161.29)
+			(xy 215.9 161.29) (xy 223.52 161.29)
 		)
 		(stroke
@@
 	(wire
 		(pts
+			(xy 336.55 147.32) (xy 336.55 153.67)
+		)
+		(stroke
+			(width 0)
+			(type default)
+		)
+	)
+	(wire
+		(pts
 			(xy 67.31 166.37) (xy 67.31 179.07)
 		)
@@
 	(wire
 		(pts
-			(xy 337.82 163.83) (xy 350.52 163.83)
+			(xy 120.65 113.03) (xy 120.65 100.33)
 		)
 		(stroke
@@
 	(wire
 		(pts
-			(xy 120.65 113.03) (xy 120.65 100.33)
+			(xy 280.67 203.2) (xy 283.21 203.2)
 		)
 		(stroke
@@
 	(wire
 		(pts
-			(xy 280.67 203.2) (xy 283.21 203.2)
+			(xy 339.09 153.67) (xy 339.09 149.86)
 		)
 		(stroke
@@
 	(wire
 		(pts
+			(xy 336.55 147.32) (xy 340.36 147.32)
+		)
+		(stroke
+			(width 0)
+			(type default)
+		)
+	)
+	(wire
+		(pts
 			(xy 212.09 119.38) (xy 215.9 119.38)
 		)
@@
 	(wire
 		(pts
+			(xy 340.36 99.06) (xy 330.2 99.06)
+		)
+		(stroke
+			(width 0)
+			(type default)
+		)
+	)
+	(wire
+		(pts
 			(xy 148.59 80.01) (xy 163.83 80.01)
 		)
@@
 	(wire
 		(pts
-			(xy 340.36 149.86) (xy 340.36 161.29)
-		)
-		(stroke
-			(width 0)
-			(type default)
-		)
-	)
-	(wire
-		(pts
 			(xy 104.14 73.66) (xy 104.14 48.26)
 		)
@@
 	(wire
 		(pts
-			(xy 353.06 161.29) (xy 353.06 170.18)
-		)
-		(stroke
-			(width 0)
-			(type default)
-		)
-	)
-	(wire
-		(pts
 			(xy 215.9 45.72) (xy 215.9 44.45)
 		)
@@
 	(wire
 		(pts
+			(xy 261.62 45.72) (xy 304.8 45.72)
+		)
+		(stroke
+			(width 0)
+			(type default)
+		)
+	)
+	(wire
+		(pts
 			(xy 281.94 182.88) (xy 281.94 200.66)
 		)
@@
 	(wire
 		(pts
-			(xy 350.52 163.83) (xy 350.52 170.18)
-		)
-		(stroke
-			(width 0)
-			(type default)
-		)
-	)
-	(wire
-		(pts
 			(xy 109.22 153.67) (xy 109.22 158.75)
 		)
@@
 	(wire
 		(pts
-			(xy 337.82 147.32) (xy 337.82 163.83)
-		)
-		(stroke
-			(width 0)
-			(type default)
-		)
-	)
-	(wire
-		(pts
 			(xy 223.52 127) (xy 212.09 127)
 		)
@@
 	(wire
 		(pts
+			(xy 325.12 41.91) (xy 325.12 101.6)
+		)
+		(stroke
+			(width 0)
+			(type default)
+		)
+	)
+	(wire
+		(pts
 			(xy 106.68 153.67) (xy 105.41 153.67)
 		)
@@
 	(wire
 		(pts
+			(xy 304.8 45.72) (xy 304.8 60.96)
+		)
+		(stroke
+			(width 0)
+			(type default)
+		)
+	)
+	(wire
+		(pts
 			(xy 212.09 48.26) (xy 212.09 85.09)
 		)
@@
 	(symbol
 		(lib_id "Connector:Conn_01x02_Pin")
-		(at 350.52 175.26 90)
+		(at 336.55 158.75 90)
 		(unit 1)
 		(exclude_from_sim no)
@@
 		(fields_autoplaced yes)
 		(property "Reference" "J19"
-			(at 354.33 173.3549 90)
+			(at 340.36 156.8449 90)
 			(effects
 				(font
@@
 		)
 		(property "Value" "Serial Pads"
-			(at 354.33 175.8949 90)
+			(at 340.36 159.3849 90)
 			(effects
 				(font
@@
 		)
 		(property "Footprint" ""
-			(at 350.52 175.26 0)
+			(at 336.55 158.75 0)
 			(effects
 				(font
@@
 		)
 		(property "Datasheet" "~"
-			(at 350.52 175.26 0)
+			(at 336.55 158.75 0)
 			(effects
 				(font
@@
 		)
 		(property "Description" "Generic connector, single row, 01x02, script generated"
-			(at 350.52 175.26 0)
+			(at 336.55 158.75 0)
 			(effects
 				(font
@@
 					(unit 1)
 				)
+			)
+		)
+	)
+	(symbol
+		(lib_id "Connector:USB_C_Plug_USB2.0")
+		(at 327.66 26.67 270)
+		(unit 1)
+		(exclude_from_sim no)
+		(in_bom yes)
+		(on_board yes)
+		(dnp no)
+		(fields_autoplaced yes)
+		(property "Reference" "P1"
+			(at 346.71 25.3999 90)
+			(effects
+				(font
+					(size 1.27 1.27)
+				)
+				(justify left)
+			)
+		)
+		(property "Value" "USB_C_Plug_USB2.0"
+			(at 346.71 27.9399 90)
+			(effects
+				(font
+					(size 1.27 1.27)
+				)
+				(justify left)
+			)
+		)
+		(property "Footprint" ""
+			(at 327.66 30.48 0)
+			(effects
+				(font
+					(size 1.27 1.27)
+				)
+				(hide yes)
+			)
+		)
+		(property "Datasheet" "https://www.usb.org/sites/default/files/documents/usb_type-c.zip"
+			(at 327.66 30.48 0)
+			(effects
+				(font
+					(size 1.27 1.27)
+				)
+				(hide yes)
+			)
+		)
+		(property "Description" "USB 2.0-only Type-C Plug connector"
+			(at 327.66 26.67 0)
+			(effects
+				(font
+					(size 1.27 1.27)
+				)
+				(hide yes)
+			)
+		)
+		(pin "A9"
+		)
+		(pin "S1"
+		)
+		(pin "A1"
+		)
+		(pin "A12"
+		)
+		(pin "B1"
+		)
+		(pin "B12"
+		)
+		(pin "A4"
+		)
+		(pin "B5"
+		)
+		(pin "B9"
+		)
+		(pin "B4"
+		)
+		(pin "A5"
+		)
+		(pin "A7"
+		)
+		(pin "A6"
+		)
+		(instances
+			(project "LumioV2"
+				(path "/3846334d-19c4-4a22-b295-63d299434ecf"
+					(reference "P1")
+					(unit 1)
+				)

Commit message: began routing
Parts:
- added C29, C30, C31, C32, C33, C36, C37: 100nF, Capacitor_SMD:C_0402_1005Metric_Pad0.74x0.62mm_HandSolder, symbol Device:C_Small
- added C34, C35: 1uF, Capacitor_SMD:C_0402_1005Metric_Pad0.74x0.62mm_HandSolder, symbol Device:C_Small
- added J20: Conn_02x13_Odd_Even, Connector_PinHeader_2.54mm:PinHeader_2x13_P2.54mm_Horizontal, symbol Connector_Generic:Conn_02x13_Odd_Even
- added J21: Conn_02x02_Odd_Even, Connector_PinHeader_2.54mm:PinHeader_2x02_P2.54mm_Vertical, symbol Connector_Generic:Conn_02x02_Odd_Even
- added R2: 5.1K, Resistor_SMD:R_0805_2012Metric_Pad1.20x1.40mm_HandSolder, symbol Device:R_Small
- added R3, R4: 27, Resistor_SMD:R_0805_2012Metric_Pad1.20x1.40mm_HandSolder, symbol Device:R_Small
- added SW1, SW2: SW_Push, Button_Switch_SMD:SW_SPST_PTS647_Sx50, symbol Switch:SW_Push
- C25, C26, C27, C28: footprint (none) -> Capacitor_SMD:C_0402_1005Metric_Pad0.74x0.62mm_HandSolder
- J19: footprint (none) -> Connector_PinHeader_2.54mm:PinHeader_1x02_P2.54mm_Vertical
- L1: footprint Inductor_THT:L_Radial_D21.0mm_P19.00mm -> Inductor_THT:L_Radial_D10.0mm_P5.00mm_Fastron_07M
- P1: footprint (none) -> Connector_USB:USB_C_Receptacle_GCT_USB4105-xx-A_16P_TopMnt_Horizontal
Connections:
- net +3V3: now also C28.1, U4.1 (IOVDD), U4.10 (IOVDD), U4.22 (IOVDD), U4.33 (IOVDD), U4.42 (IOVDD), U4.43 (ADC_AVDD), U4.44 (VREG_VIN), U4.48 (USB_VDD), U4.49 (IOVDD), C29.1, C30.1, C31.1, C32.1, C33.1, C34.2
- net +5V: now also P1.A4 (VBUS), P1.A9 (VBUS), P1.B4 (VBUS), P1.B9 (VBUS)
- net GND: now also C28.2, P1.S1 (SHIELD), U4.19 (TESTEN), C29.2, C30.2, C31.2, C32.2, C33.2, C34.1, C35.1, C36.1, C37.1, R2.2, SW1.1, SW2.1; no longer C28.1
- net at U4.56 (~{QSPI_SS}), U5.1 (/CS): now also SW2.2
- net at U4.11 (GPIO8): now also J20.9 (Pin_9)
- net at U4.12 (GPIO9): now also J20.10 (Pin_10)
- net at U4.13 (GPIO10): now also J20.11 (Pin_11)
- net at U4.14 (GPIO11): now also J20.12 (Pin_12)
- net at U4.15 (GPIO12): now also J20.13 (Pin_13)
- net at U4.16 (GPIO13): now also J20.14 (Pin_14)
- net at U4.17 (GPIO14): now also J20.15 (Pin_15)
- net at U4.18 (GPIO15): now also J20.16 (Pin_16)
- net at U4.2 (GPIO0): now also J20.1 (Pin_1)
- net +1V1: now reaches U4.23 (DVDD), U4.50 (DVDD)
- net +1V1: now also U4.45 (VREG_VOUT), C35.2, C36.2, C37.2
- net at U4.26 (RUN): now also SW1.2
- net at U4.27 (GPIO16): now also J20.17 (Pin_17)
- net at U4.28 (GPIO17): now also J20.18 (Pin_18)
- net at U4.29 (GPIO18): now also J20.19 (Pin_19)
- net at U4.3 (GPIO1): now also J20.2 (Pin_2)
- net at U4.30 (GPIO19): now also J20.20 (Pin_20)
- net at U4.31 (GPIO20): now also J20.21 (Pin_21)
- net at U4.32 (GPIO21): now also J20.22 (Pin_22)
- net at U4.34 (GPIO22): now also J20.23 (Pin_23)
- net at U4.35 (GPIO23): now also J20.24 (Pin_24)
- net at U4.36 (GPIO24): now also J20.25 (Pin_25)
- net at U4.37 (GPIO25): now also J20.26 (Pin_26)
- net at U4.38 (GPIO26/ADC0): now also J21.1 (Pin_1)
- net at U4.39 (GPIO27/ADC1): now also J21.2 (Pin_2)
- net at U4.4 (GPIO2): now also J20.3 (Pin_3)
- net at U4.40 (GPIO28/ADC2): now also J21.3 (Pin_3)
- net at U4.41 (GPIO29/ADC3): now also J21.4 (Pin_4)
- net at U4.46 (USB_DM): now also R3.2; no longer P1.A7 (D-)
- net at U4.47 (USB_DP): now also R4.1; no longer P1.A6 (D+)
- net at U4.5 (GPIO3): now also J20.4 (Pin_4)
- net at U4.51 (QSPI_SD3): now also U5.7 (/HOLD_or_/RESET_(IO3))
- net at U4.54 (QSPI_SD2): now also U5.3 (/WP_(IO2))
- net at U4.6 (GPIO4): now also J20.5 (Pin_5)
- net at U4.7 (GPIO5): now also J20.6 (Pin_6)
- net at U4.8 (GPIO6): now also J20.7 (Pin_7)
- net at U4.9 (GPIO7): now also J20.8 (Pin_8)
- net at P1.A5 (CC): now also R2.1
- new net: C25.2, U5.8 (VCC)
- new net USB_N: P1.A7 (D-), R3.1
- new net USB_P: P1.A6 (D+), R4.2
- no-connect marks 18 -> 19
Other:
- note added: "make sure close to pin 44"
- note added: "make sure close to pin 45"
- moved on the sheet: C25, C26, C27, J19, P1, U4, U5, Y1
