File: LumioV2.kicad_sch (KiCad schematic)
At the start: 79 parts, among them J1 I2C POINT 1 - QWIIC, J10 MOTOR B, J11 Analog Input, J12 Analog Input, J13 Analog Input, J14 Analog Input, J15 Analog Input, J16 Analog Input, J17 Analog Input, J18 Analog Input, J19 Serial Pads, J2 I2C POINT 2 - QWIIC, J20 Conn_02x13_Odd_Even, J21 Conn_02x02_Odd_Even, J3 I2C POINT 3 - JST-PH, J4 I2C POINT 4 - JST-PH, J5 Raspi 5, J6 US Dist - Front, J7 US Dist - Back, J8 USB_C_Receptacle_USB2.0_14P, J9 MOTOR A, SW1 SW_Push, SW2 SW_Push, U1 LM2577T-ADJ/NOPB, U2 L298N, U3 MCP3008, U4 RP2040, U5 W25Q64JVXGIQ TR, Y1 Crystal, Y2 ECS-2520MV-xxx-xx

Commit message: routed abit; replaced the MCP3008 footprint to a 16 pin socket, so that i can swap it easily if the user fries it somehow
Parts:
- removed J19: Serial Pads, Connector_PinHeader_2.54mm:PinHeader_1x02_P2.54mm_Vertical, symbol Connector:Conn_01x02_Pin
- removed Y1: Crystal, Crystal:Crystal_SMD_HC49-SD, symbol Device:Crystal
- added J20: Header programmer, Connector_PinHeader_2.54mm:PinHeader_2x02_P2.54mm_Vertical, symbol Connector_Generic:Conn_02x02_Counter_Clockwise
- added R6: 1K, Resistor_SMD:R_0603_1608Metric, symbol Device:R_Small
- C40: renamed from C26; value 33pF -> 15pF
- C41: renamed from C27; value 33pF -> 15pF
- J2: renamed from J8; footprint Connector_USB:USB_C_Receptacle_Amphenol_12401610E4-2A -> Connector_USB:USB_C_Receptacle_G-Switch_GT-USB-7010ASV
- R1: renamed from R6; footprint Resistor_SMD:R_0805_2012Metric_Pad1.20x1.40mm_HandSolder -> Resistor_SMD:R_0603_1608Metric
- R2: renamed from R5; footprint Resistor_SMD:R_0805_2012Metric_Pad1.20x1.40mm_HandSolder -> Resistor_SMD:R_0603_1608Metric
- R4: renamed from R3; footprint Resistor_SMD:R_0805_2012Metric_Pad1.20x1.40mm_HandSolder -> Resistor_SMD:R_0603_1608Metric
- R5: renamed from R4; footprint Resistor_SMD:R_0805_2012Metric_Pad1.20x1.40mm_HandSolder -> Resistor_SMD:R_0603_1608Metric
- U4: renamed from U3; footprint Package_SO:SOIC-16_3.9x9.9mm_P1.27mm -> Package_DIP:DIP-16_W7.62mm_Socket_LongPads
- U5: renamed from U4; private KLC_S4.2_VREG_VOUT -> (none)
- renumbered C19 to C1, C35 to C10, C20 to C16, C13 to C17, C31 to C18, C36 to C19, C18 to C2, C7 to C20, C34 to C21, C37 to C22, C14 to C23, C28 to C24, C11 to C25, C12 to C26, C10 to C27, C33 to C28, C2 to C3, C6 to C30, C30 to C31, C8 to C32, C15 to C33, C21 to C34, C32 to C35, C9 to C36, C25 to C37, C3 to C4, C1 to C5, C4 to C6, C5 to C7, C16 to C8, C17 to C9, D5 to D1, D1 to D2, D8 to D3, D9 to D5, D3 to D6, D6 to D8, D2 to D9, J5 to J1, J11 to J10, J15 to J11, J14 to J13, J17 to J14, J16 to J15, J13 to J16, J18 to J17, J7 to J18, J6 to J19, J20 to J3, J3 to J5, J2 to J6, J1 to J7, J10 to J8, R1 to R3, SW2 to SW1, SW1 to SW2, U5 to U3, Y2 to Y1
Connections:
- net +3V3: now also C37.2, U3.8 (VCC)
- net GND: now also Y1.2 (GND), Y1.4 (VDD)
- net at J1.18 (Pin_18): now also J20.1 (Pin_1)
- net at J1.22 (Pin_22): now also J20.2 (Pin_2)
- net at C41.1, U5.20 (XIN): now also Y1.3 (OUT)
- net at U5.21 (XOUT): now also R6.1; no longer C40.2
- net at U5.24 (SWCLK): now also J20.3 (Pin_3)
- net at U5.25 (SWDIO): now also J20.4 (Pin_4)
- net at Y1.1 (Tri-State): now also C40.2, R6.2
Other:
- moved on the sheet: C40, C41, Y1
