File: Hardware/LumioV2.kicad_pcb (KiCad board)
At the start: 4 copper layers, 117.5 x 73 mm, 79 parts, among them J1 Raspi 5, J10 Analog Input, J11 Analog Input, J12 Header programmer, J13 MOTOR B, J14 USB_C_Receptacle_USB2.0_14P, J15 Conn_02x13_Odd_Even, J16 US Dist - Front, J17 US Dist - Back, J18 Sensor power lines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

Commit message: resolved bugs, added documentation, and created filled zone for 3v3 on B.Cu and connected to 3v pins on raspi
Parts:
- added C9: 100nF, Capacitor_SMD:C_0402_1005Metric_Pad0.74x0.62mm_HandSolder, F.Cu at (67.6, 60.4)
Routing:
- net +3V3: track 415.8 -> 504.4 mm, vias 5 -> 9
- net GND: track 76.9 -> 80.5 mm, vias 21 -> 33
- net Net-(U5-XOUT): track 7.26 -> 9.08 mm
- net Net-(U5-XIN): track 8.96 -> 8.33 mm
- net Net-(U3-/WP_(IO2)): track 15.4 -> 14.9 mm
- net (no net): vias 1 -> 0
- added copper zone on B.Cu, net +3V3
- added copper zone on In1.Cu, net +3V3
